Commit message: add T108 new type support

File: tianracer_description/urdf/tianracer_compact.urdf (robot description, URDF)
Before this commit: robot tianracer_description, 10 links, 9 joints
Links:
- removed link camera
- added link base_footprint
- added link camera_link, mass 0.020388; collision mesh filename=package://tianracer_description/meshes/camera.STL; visual mesh filename=package://tianracer_description/meshes/camera.STL
- added link imu_link
- link base_link: mass None -> 1.0055
Joints:
- added joint base_footprint_to_base_link: type fixed, parent base_footprint, child base_link, origin xyz=0 0 0.0315 rpy=0 0 0
- added joint base_link_to_imu: type fixed, parent base_link, child imu_link, origin xyz=0.22 0 0.1 rpy=0 0 0
- joint camera_joint: child camera -> camera_link
