Commit message: feat: tianracer nav in sim

File: tianracer_gazebo/urdf/tianracer.xacro (robot description, xacro)
@@ -11,6 +11,6 @@
       </geometry>
       <origin xyz="-0.13 0 0" rpy="0 0 0" />
-      <material name="yellow">
-        <color rgba="0.8 0.3 0.1 0.5" />
+      <material name="gray">
+        <color rgba="0.5 0.5 0.5 1.0" />
       </material>
     </visual>
