Commit message: style:delete file with redundant name _02 for the same functionality

File: tianracer_gazebo/urdf/macros.xacro (robot description, xacro)
@@ -3,5 +3,5 @@
 <!-- transmission macros -->
 <xacro:macro name="wheel_transmission" params="name">
-  <transmission name="${name}_transmission" type="SimpleTransmission">
+  <transmission name="${tf_prefix}_${name}_transmission" type="SimpleTransmission">
     <type>transmission_interface/SimpleTransmission</type>
     <joint name="${name}_joint">
@@ -15,5 +15,5 @@
 </xacro:macro>
 <xacro:macro name="steering_hinge_transmission" params="name">
-  <transmission name="${name}_transmission" type="SimpleTransmission">
+  <transmission name="${tf_prefix}_${name}_transmission" type="SimpleTransmission">
     <type>transmission_interface/SimpleTransmission</type>
     <joint name="${name}_joint">

File: tianracer_gazebo/urdf/tianracer.xacro (robot description, xacro)
@@ -1,8 +1,8 @@
 <?xml version="1.0" encoding="utf-8"?>
-<robot name="tianracer" xmlns:xacro="http://www.ros.org/wiki/xacro">
+<robot xmlns:xacro="http://www.ros.org/wiki/xacro">
   <xacro:include filename="$(find tianracer_gazebo)/urdf/macros.xacro" />
-  <link name="base_footprint">
-  </link>
-  <link name="base_link">
+  <link name="${tf_prefix}base_footprint">
+  </link>
+  <link name="${tf_prefix}base_link">
     <visual>
       <geometry>
@@ -23,9 +23,9 @@
   </link>
   <joint name="base_link2base_footprint" type="fixed">
-    <parent link="base_footprint" />
-    <child link="base_link" />
+    <parent link="${tf_prefix}base_footprint" />
+    <child link="${tf_prefix}base_link" />
     <origin xyz="0 0 0.032" rpy="0 0 0" />
   </joint>
-  <link name="base_inertia">
+  <link name="${tf_prefix}base_inertia">
     <inertial>
       <origin xyz="0 0 0" />
@@ -36,8 +36,8 @@
   <joint name="chassis_inertia_joint" type="fixed">
     <origin xyz="0 0 0" rpy="0 0 0" />
-    <parent link="base_link" />
-    <child link="base_inertia" />
-  </joint>
-  <link name="left_steering_hinge">
+    <parent link="${tf_prefix}base_link" />
+    <child link="${tf_prefix}base_inertia" />
+  </joint>
+  <link name="${tf_prefix}left_steering_hinge">
     <visual>
       <geometry>
@@ -64,12 +64,12 @@
   </link>
   <joint name="left_steering_hinge_joint" type="revolute">
-    <parent link="base_link" />
-    <child link="left_steering_hinge" />
+    <parent link="${tf_prefix}base_link" />
+    <child link="${tf_prefix}left_steering_hinge" />
     <origin xyz="0.13 0.065 0" />
     <axis xyz="0 0 1" />
     <limit lower="-0.6" upper="0.6" effort="5.0" velocity="1000.0" />
   </joint>
-  <xacro:steering_hinge_transmission name="left_steering_hinge" />
-  <link name="left_front_wheel">
+  <xacro:steering_hinge_transmission name="left_steering_hinge"/>
+  <link name="${tf_prefix}left_front_wheel">
     <visual>
       <geometry>
@@ -94,12 +94,12 @@
   </link>
   <joint name="left_front_wheel_joint" type="continuous">
-    <parent link="left_steering_hinge" />
-    <child link="left_front_wheel" />
+    <parent link="${tf_prefix}left_steering_hinge" />
+    <child link="${tf_prefix}left_front_wheel" />
     <origin xyz="0 0.025 0" />
     <axis xyz="0 1 0" />
     <limit effort="10" velocity="1000" />
   </joint>
-  <xacro:wheel_transmission name="left_front_wheel" />
-  <link name="right_steering_hinge">
+  <xacro:wheel_transmission name="left_front_wheel"/>
+  <link name="${tf_prefix}right_steering_hinge">
     <visual>
       <geometry>
@@ -124,12 +124,12 @@
   </link>
   <joint name="right_steering_hinge_joint" type="revolute">
-    <parent link="base_link" />
-    <child link="right_steering_hinge" />
+    <parent link="${tf_prefix}base_link" />
+    <child link="${tf_prefix}right_steering_hinge" />
     <origin xyz="0.13 -0.065 0" />
     <axis xyz="0 0 1" />
     <limit lower="-0.6" upper="0.6" effort="5.0" velocity="1000.0" />
   </joint>
-  <xacro:steering_hinge_transmission name="right_steering_hinge" />
-  <link name="right_front_wheel">
+  <xacro:steering_hinge_transmission name="right_steering_hinge"/>
+  <link name="${tf_prefix}right_front_wheel">
     <visual>
       <geometry>
@@ -154,12 +154,12 @@
   </link>
   <joint name="right_front_wheel_joint" type="continuous">
-    <parent link="right_steering_hinge" />
-    <child link="right_front_wheel" />
+    <parent link="${tf_prefix}right_steering_hinge" />
+    <child link="${tf_prefix}right_front_wheel" />
     <origin xyz="0 -0.025 0" />
     <axis xyz="0 1 0" />
     <limit effort="10" velocity="1000" />
   </joint>
-  <xacro:wheel_transmission name="right_front_wheel" />
-  <link name="left_rear_wheel">
+  <xacro:wheel_transmission name="right_front_wheel"/>
+  <link name="${tf_prefix}left_rear_wheel">
     <visual>
       <geometry>
@@ -184,12 +184,12 @@
   </link>
   <joint name="left_rear_wheel_joint" type="continuous">
-    <parent link="base_link" />
-    <child link="left_rear_wheel" />
+    <parent link="${tf_prefix}base_link" />
+    <child link="${tf_prefix}left_rear_wheel" />
     <origin xyz="-0.13 0.09 0" />
     <axis xyz="0 1 0" />
     <limit effort="10" velocity="1000" />
   </joint>
-  <xacro:wheel_transmission name="left_rear_wheel" />
-  <link name="right_rear_wheel">
+  <xacro:wheel_transmission name="left_rear_wheel"/>
+  <link name="${tf_prefix}right_rear_wheel">
     <visual>
       <geometry>
@@ -214,12 +214,12 @@
   </link>
   <joint name="right_rear_wheel_joint" type="continuous">
-    <parent link="base_link" />
-    <child link="right_rear_wheel" />
+    <parent link="${tf_prefix}base_link" />
+    <child link="${tf_prefix}right_rear_wheel" />
     <origin xyz="-0.13 -0.09 0" />
     <axis xyz="0 1 0" />
     <limit effort="10" velocity="1000" />
   </joint>
-  <xacro:wheel_transmission name="right_rear_wheel" />
-  <link name="camera">
+  <xacro:wheel_transmission name="right_rear_wheel"/>
+  <link name="${tf_prefix}camera">
     <visual>
       <geometry>
@@ -245,10 +245,10 @@
   </link>
   <joint name="camera_joint" type="fixed">
-    <parent link="base_link" />
-    <child link="camera" />
+    <parent link="${tf_prefix}base_link" />
+    <child link="${tf_prefix}camera" />
     <origin xyz="0.14851 0.0022137 0.0975" />
     <axis xyz="0 0 1" />
   </joint>
-  <link name="real_sense">
+  <link name="${tf_prefix}real_sense">
     <visual>
       <geometry>
@@ -274,16 +274,16 @@
   </link>
   <joint name="realsense_joint" type="fixed">
-    <parent link="base_link" />
-    <child link="real_sense" />
+    <parent link="${tf_prefix}base_link" />
+    <child link="${tf_prefix}real_sense" />
     <origin xyz="0.18864 0.0038046 0.052021" />
     <axis xyz="0 0 1" />
   </joint>
-  <link name="realsense_depth" />
+  <link name="${tf_prefix}realsense_depth" />
   <joint name="realsense_depth_joint" type="fixed">
     <origin xyz="0 0 0" rpy="-1.5708 0 -1.5708" />
-    <parent link="real_sense" />
-    <child link="realsense_depth" />
-  </joint>
-  <link name="laser">
+    <parent link="${tf_prefix}real_sense" />
+    <child link="${tf_prefix}realsense_depth" />
+  </joint>
+  <link name="${tf_prefix}laser">
     <visual>
       <geometry>
@@ -309,10 +309,10 @@
   </link>
   <joint name="laser_joint" type="fixed">
-    <parent link="base_link" />
-    <child link="laser" />
+    <parent link="${tf_prefix}base_link" />
+    <child link="${tf_prefix}laser" />
     <origin xyz="0.093603 0 0.12377" />
     <axis xyz="0 0 1" />
   </joint>
-  <link name="imu">
+  <link name="${tf_prefix}imu">
     <visual>
       <geometry>
@@ -337,6 +337,6 @@
   </link>
   <joint name="imu_joint" type="fixed">
-    <parent link="base_link" />
-    <child link="imu" />
+    <parent link="${tf_prefix}base_link" />
+    <child link="${tf_prefix}imu" />
     <origin xyz="0 0 0.02" />
     <axis xyz="0 0 1" />

File: tianracer_gazebo/urdf/tianracer_run.xacro (robot description, xacro)
@@ -8,5 +8,5 @@
     <xacro:property name="tf_prefix" value="${prefix}/" />
     </xacro:unless>
-    <xacro:include filename="$(find tianracer_gazebo)/urdf/tianracer.urdf.xacro" />
+    <xacro:include filename="$(find tianracer_gazebo)/urdf/tianracer.xacro" />
     <tianbot_mini/>
 </robot>
